File: step-up.kicad_sch (KiCad schematic)
At the start: 7 parts, among them U1 MT3608

Commit message: terminando, aun falta una ultima revision previa a la fabricacion
Parts:
- added R11: 20K, Resistor_SMD:R_0603_1608Metric, symbol Device:R
- C1: footprint Capacitor_SMD:C_0603_1608Metric -> Capacitor_SMD:C_1206_3216Metric
- C2: footprint Capacitor_SMD:C_0805_2012Metric_Pad1.18x1.45mm_HandSolder -> Capacitor_SMD:C_1206_3216Metric
- D1: footprint Diode_SMD:D_SOD-123 -> Diode_SMD:D_SMB
- L1: footprint MSS_Devices:L_Bourns_SDR0403 -> MSS_Devices:L_Bourns-SDE0805A_7x7.8mm
- R1: value R -> 22K
- U1: value MT3608 -> SDB628
Connections:
- net VOUT_12V: now also R11.1; no longer R1.1
- new net: R1.1, R11.2
Other:
- note added: "Vo=0.6x[1+((R1+R11)/R2)]"
- moved on the sheet: R1, R2
Changed lines of the file:
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@@
     (rev "v1.0.0")
   )
+  (junction (at 156.21 80.01) (diameter 0) (color 0 0 0 0)
+  )
   (junction (at 115.57 95.25) (diameter 0) (color 0 0 0 0)
   )
@@
   (junction (at 142.24 80.01) (diameter 0) (color 0 0 0 0)
   )
-  (junction (at 156.21 80.01) (diameter 0) (color 0 0 0 0)
-  )
-  (junction (at 156.21 95.25) (diameter 0) (color 0 0 0 0)
+  (junction (at 156.21 100.33) (diameter 0) (color 0 0 0 0)
   )
   (junction (at 115.57 80.01) (diameter 0) (color 0 0 0 0)
@@
     (stroke (width 0) (type default) (color 0 0 0 0))
   )
-  (wire (pts (xy 156.21 95.25) (xy 156.21 97.79))
-    (stroke (width 0) (type default) (color 0 0 0 0))
-  )
-  (wire (pts (xy 137.16 100.33) (xy 147.32 100.33))
+  (wire (pts (xy 156.21 100.33) (xy 156.21 105.41))
+    (stroke (width 0) (type default) (color 0 0 0 0))
+  )
+  (wire (pts (xy 137.16 100.33) (xy 156.21 100.33))
     (stroke (width 0) (type default) (color 0 0 0 0))
   )
@@
     (stroke (width 0) (type default) (color 0 0 0 0))
   )
-  (wire (pts (xy 147.32 95.25) (xy 156.21 95.25))
-    (stroke (width 0) (type default) (color 0 0 0 0))
-  )
   (wire (pts (xy 142.24 80.01) (xy 142.24 95.25))
     (stroke (width 0) (type default) (color 0 0 0 0))
   )
-  (wire (pts (xy 156.21 95.25) (xy 156.21 92.71))
-    (stroke (width 0) (type default) (color 0 0 0 0))
-  )
-  (wire (pts (xy 147.32 100.33) (xy 147.32 95.25))
-    (stroke (width 0) (type default) (color 0 0 0 0))
-  )
-  (wire (pts (xy 156.21 105.41) (xy 156.21 106.68))
+  (wire (pts (xy 156.21 90.17) (xy 156.21 91.44))
+    (stroke (width 0) (type default) (color 0 0 0 0))
+  )
+  (wire (pts (xy 156.21 100.33) (xy 156.21 99.06))
+    (stroke (width 0) (type default) (color 0 0 0 0))
+  )
+  (wire (pts (xy 156.21 113.03) (xy 156.21 115.57))
     (stroke (width 0) (type default) (color 0 0 0 0))
   )
@@
     (stroke (width 0) (type default) (color 0 0 0 0))
   )
-  (wire (pts (xy 156.21 80.01) (xy 152.4 80.01))
-    (stroke (width 0) (type default) (color 0 0 0 0))
-  )
-  (wire (pts (xy 156.21 85.09) (xy 156.21 80.01))
+  (wire (pts (xy 156.21 80.01) (xy 156.21 82.55))
     (stroke (width 0) (type default) (color 0 0 0 0))
   )
@@
     (stroke (width 0) (type default) (color 0 0 0 0))
   )
-  (wire (pts (xy 166.37 80.01) (xy 156.21 80.01))
+  (wire (pts (xy 152.4 80.01) (xy 156.21 80.01))
     (stroke (width 0) (type default) (color 0 0 0 0))
   )
@@
     (stroke (width 0) (type default) (color 0 0 0 0))
   )
+  (wire (pts (xy 156.21 80.01) (xy 166.37 80.01))
+    (stroke (width 0) (type default) (color 0 0 0 0))
+  )
   (wire (pts (xy 166.37 91.44) (xy 166.37 80.01))
     (stroke (width 0) (type default) (color 0 0 0 0))
@@
   (wire (pts (xy 115.57 111.76) (xy 115.57 114.3))
     (stroke (width 0) (type default) (color 0 0 0 0))
+  )
+  (text "Vo=0.6x[1+((R1+R11)/R2)]" (at 158.75 72.39 0)
+    (effects (font (size 1.27 1.27)) (justify left bottom))
   )
   (text "Mt3608" (at 128.27 34.29 0)
@@
       (effects (font (size 1.27 1.27)) (justify left))
     )
-    (property "Footprint" "Capacitor_SMD:C_0805_2012Metric_Pad1.18x1.45mm_HandSolder" (id 2) (at 167.3352 99.06 0)
+    (property "Footprint" "Capacitor_SMD:C_1206_3216Metric" (id 2) (at 167.3352 99.06 0)
       (effects (font (size 1.27 1.27)) hide)
     )
@@
     (property "Reference" "D1" (id 0) (at 148.9075 73.66 0))
     (property "Value" "SS34" (id 1) (at 148.9075 76.2 0))
-    (property "Footprint" "Diode_SMD:D_SOD-123" (id 2) (at 148.59 80.01 0)
+    (property "Footprint" "Diode_SMD:D_SMB" (id 2) (at 148.59 80.01 0)
       (effects (font (size 1.27 1.27)) hide)
     )
@@
       (effects (font (size 1.27 1.27)) (justify left))
     )
-    (property "Footprint" "Capacitor_SMD:C_0603_1608Metric" (id 2) (at 116.5352 111.76 0)
+    (property "Footprint" "Capacitor_SMD:C_1206_3216Metric" (id 2) (at 116.5352 111.76 0)
       (effects (font (size 1.27 1.27)) hide)
     )
@@
     (property "Reference" "L1" (id 0) (at 129.54 73.66 90))
     (property "Value" "22uH" (id 1) (at 129.54 76.2 90))
-    (property "Footprint" "MSS_Devices:L_Bourns_SDR0403" (id 2) (at 129.54 80.01 0)
+    (property "Footprint" "MSS_Devices:L_Bourns-SDE0805A_7x7.8mm" (id 2) (at 129.54 80.01 0)
       (effects (font (size 1.27 1.27)) hide)
     )
@@
     (pin "2")
   )
-  (symbol (lib_id "Device:R") (at 156.21 101.6 0) (unit 1)
-    (in_bom yes) (on_board yes) (fields_autoplaced)
-    (property "Reference" "R2" (id 0) (at 158.75 100.3299 0)
-      (effects (font (size 1.27 1.27)) (justify left))
-    )
-    (property "Value" "2.2k" (id 1) (at 158.75 102.8699 0)
-      (effects (font (size 1.27 1.27)) (justify left))
-    )
-    (property "Footprint" "Resistor_SMD:R_0603_1608Metric" (id 2) (at 154.432 101.6 90)
-      (effects (font (size 1.27 1.27)) hide)
-    )
-    (property "Datasheet" "~" (id 3) (at 156.21 101.6 0)
-      (effects (font (size 1.27 1.27)) hide)
-    )
-    (pin "1")
-    (pin "2")
-  )
-  (symbol (lib_id "Device:R") (at 156.21 88.9 0) (unit 1)
-    (in_bom yes) (on_board yes) (fields_autoplaced)
-    (property "Reference" "R1" (id 0) (at 158.75 87.6299 0)
-      (effects (font (size 1.27 1.27)) (justify left))
-    )
-    (property "Value" "R" (id 1) (at 158.75 90.1699 0)
-      (effects (font (size 1.27 1.27)) (justify left))
-    )
-    (property "Footprint" "Resistor_SMD:R_0603_1608Metric" (id 2) (at 154.432 88.9 90)
-      (effects (font (size 1.27 1.27)) hide)
-    )
-    (property "Datasheet" "~" (id 3) (at 156.21 88.9 0)
+  (symbol (lib_id "Device:R") (at 156.21 109.22 0) (unit 1)
+    (in_bom yes) (on_board yes) (fields_autoplaced)
+    (property "Reference" "R2" (id 0) (at 158.75 107.9499 0)
+      (effects (font (size 1.27 1.27)) (justify left))
+    )
+    (property "Value" "2.2k" (id 1) (at 158.75 110.4899 0)
+      (effects (font (size 1.27 1.27)) (justify left))
+    )
+    (property "Footprint" "Resistor_SMD:R_0603_1608Metric" (id 2) (at 154.432 109.22 90)
+      (effects (font (size 1.27 1.27)) hide)
+    )
+    (property "Datasheet" "~" (id 3) (at 156.21 109.22 0)
+      (effects (font (size 1.27 1.27)) hide)
+    )
+    (pin "1")
+    (pin "2")
+  )
+  (symbol (lib_id "Device:R") (at 156.21 86.36 0) (unit 1)
+    (in_bom yes) (on_board yes) (fields_autoplaced)
+    (property "Reference" "R11" (id 0) (at 158.75 85.0899 0)
+      (effects (font (size 1.27 1.27)) (justify left))
+    )
+    (property "Value" "20K" (id 1) (at 158.75 87.6299 0)
+      (effects (font (size 1.27 1.27)) (justify left))
+    )
+    (property "Footprint" "Resistor_SMD:R_0603_1608Metric" (id 2) (at 154.432 86.36 90)
+      (effects (font (size 1.27 1.27)) hide)
+    )
+    (property "Datasheet" "~" (id 3) (at 156.21 86.36 0)
+      (effects (font (size 1.27 1.27)) hide)
+    )
+    (pin "1")
+    (pin "2")
+  )
+  (symbol (lib_id "Device:R") (at 156.21 95.25 0) (unit 1)
+    (in_bom yes) (on_board yes) (fields_autoplaced)
+    (property "Reference" "R1" (id 0) (at 158.75 93.9799 0)
+      (effects (font (size 1.27 1.27)) (justify left))
+    )
+    (property "Value" "22K" (id 1) (at 158.75 96.5199 0)
+      (effects (font (size 1.27 1.27)) (justify left))
+    )
+    (property "Footprint" "Resistor_SMD:R_0603_1608Metric" (id 2) (at 154.432 95.25 90)
+      (effects (font (size 1.27 1.27)) hide)
+    )
+    (property "Datasheet" "~" (id 3) (at 156.21 95.25 0)
       (effects (font (size 1.27 1.27)) hide)
     )
@@
     (in_bom yes) (on_board yes) (fields_autoplaced)
     (property "Reference" "U1" (id 0) (at 129.54 87.63 0))
-    (property "Value" "MT3608" (id 1) (at 129.54 90.17 0))
+    (property "Value" "SDB628" (id 1) (at 129.54 90.17 0))
     (property "Footprint" "Package_TO_SOT_SMD:SOT-23-6" (id 2) (at 130.81 104.14 0)
       (effects (font (size 1.27 1.27) italic) (justify left) hide)
     )
-    (property "Datasheet" "https://www.olimex.com/Products/Breadboarding/BB-PWR-3608/resources/MT3608.pdf" (id 3) (at 123.19 86.36 0)
+    (property "Datasheet" "https://www.uugear.com/doc/datasheet/SDB628.pdf" (id 3) (at 123.19 86.36 0)
       (effects (font (size 1.27 1.27)) hide)
     )
@@
     (pin "6")
   )
-  (symbol (lib_id "power:GND") (at 156.21 106.68 0) (unit 1)
-    (in_bom yes) (on_board yes) (fields_autoplaced)
-    (property "Reference" "#PWR013" (id 0) (at 156.21 113.03 0)
-      (effects (font (size 1.27 1.27)) hide)
-    )
-    (property "Value" "~" (id 1) (at 156.21 111.76 0))
-    (property "Footprint" "" (id 2) (at 156.21 106.68 0)
-      (effects (font (size 1.27 1.27)) hide)
-    )
-    (property "Datasheet" "" (id 3) (at 156.21 106.68 0)
-      (effects (font (size 1.27 1.27)) hide)
-    )
+  (symbol (lib_id "power:GND") (at 156.21 115.57 0) (unit 1)
+    (in_bom yes) (on_board yes) (fields_autoplaced)
+    (property "Reference" "#PWR013" (id 0) (at 156.21 121.92 0)
+      (effects (font (size 1.27 1.27)) hide)
+    )
+    (property "Value" "~" (id 1) (at 156.21 120.65 0))
+    (property "Footprint" "" (id 2) (at 156.21 115.57 0)
+      (effects (font (size 1.27 1.27)) hide)
+    )
+    (property "Datasheet" "" (id 3) (at 156.21 115.57 0)
+      (effects (font (size 1.27 1.27)) hide)
+    )
