File: gpsOled.kicad_pcb (KiCad board)
At the start: 2 copper layers, 40 x 100 mm, 55 parts, among them J1 USB_B_Micro, J2 Conn_01x02, J3 Conn_01x03, J4 SSD1306, J5 RJ45, J6 Conn_01x04, Q1 FS8205A, SW1 on/off, SW4 SW_Push, U1 MT3608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

Commit message: terminando, aun falta una ultima revision previa a la fabricacion
Parts:
- added R11: 20K, Resistor_SMD:R_0603_1608Metric, B.Cu at (160.6, 72.3)
- added R12: 2.2k, Resistor_SMD:R_0603_1608Metric, F.Cu at (161.9, 137.6)
- added kibuzzard-627F1822: G***, kibuzzard-627F1822, B.Cu at (155.3, 93.1)
- C1: footprint Capacitor_SMD:C_0603_1608Metric -> Capacitor_SMD:C_1206_3216Metric
- C2: footprint Capacitor_SMD:C_0805_2012Metric_Pad1.18x1.45mm_HandSolder -> Capacitor_SMD:C_1206_3216Metric
- C8: value ~ -> 22uF; footprint Capacitor_SMD:C_0603_1608Metric -> Capacitor_SMD:C_1206_3216Metric
- C9: value ~ -> 22uF; footprint Capacitor_SMD:C_0805_2012Metric_Pad1.18x1.45mm_HandSolder -> Capacitor_SMD:C_1206_3216Metric
- D1: footprint Diode_SMD:D_SOD-123 -> Diode_SMD:D_SMB
- D4: value ~ -> SS34; footprint Diode_SMD:D_SOD-123 -> Diode_SMD:D_SMB
- H1, H2: footprint MountingHole:MountingHole_3.2mm_M3_DIN965_Pad -> MountingHole:MountingHole_3.2mm_M3_DIN965
- H3: footprint MountingHole:MountingHole_3.2mm_M3_DIN965_Pad -> MountingHole:MountingHole_3.2mm_M3
- J2: footprint Connector_PinHeader_2.54mm:PinHeader_1x02_P2.54mm_Vertical -> Connector_PinHeader_1.27mm:PinHeader_1x02_P1.27mm_Vertical
- J5: footprint Connector_RJ:RJ45_Amphenol_54602-x08_Horizontal -> MSS_Connector:RJ45_GEN_ZQP_Horizontal
- L1: footprint MSS_Devices:L_Bourns_SDR0403 -> MSS_Devices:L_Bourns-SDE0805A_7x7.8mm
- L2: value ~ -> 22uH; footprint MSS_Devices:L_Bourns_SDR0403 -> MSS_Devices:L_Bourns-SDE0805A_7x7.8mm
- R1: value R -> 22K
- R8: value ~ -> 10K
- R9: value ~ -> 6.2K
- SW1: footprint Button_Switch_THT:SW_CuK_JS202011AQN_DPDT_Angled -> Button_Switch_SMD:SW_SPDT_PCM12
- SW2, SW3, SW4, SW5: footprint Button_Switch_SMD:SW_SPST_PTS645 -> MSS_Devices:TL3301AF160QG
- U1: value MT3608 -> SDB628
- U6: value MIC2251 -> SDB628; footprint Package_TO_SOT_SMD:SOT-23-5 -> Package_TO_SOT_SMD:SOT-23-6
- U7: footprint Package_SO:SSOP-20_3.9x8.7mm_P0.635mm -> Package_SO:SOIC-16_4.55x10.3mm_P1.27mm
- moved C8 12.9 mm to (156.8, 136.9)
- moved L1 11.8 mm to (149.4, 70.9), turned to 90 degrees
- moved R1 11.7 mm to (162.4, 73.4), turned to -90 degrees
- moved R8 10.6 mm to (161.0, 135.2)
- moved R2 10.2 mm to (161.5, 75.9), turned to 180 degrees
- moved R9 9.48 mm to (160.2, 137.6), turned to -90 degrees
- moved C1 8.17 mm to (157.2, 76.5), turned to 0 degrees
- moved D1 7.79 mm to (157.7, 67.9), turned to 180 degrees
- moved C2 7.16 mm to (162.8, 69.3), turned to -90 degrees
- moved U6 6.84 mm to (156.6, 140.6), turned to 180 degrees
- moved D4 5.95 mm to (162.5, 145.6), turned to -90 degrees
- moved C9 4.62 mm to (161.7, 140.6), turned to 180 degrees
- moved SW1 3.25 mm to (164.1, 93.9)
- moved L2 2.80 mm to (155.6, 147.8), turned to 0 degrees
- moved U1 2.59 mm to (157.4, 72.7), turned to 180 degrees
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Connections:
- R1 pad 1: +12V -> Net-(R1-Pad1)
- R9 pad 2: GND -> Net-(R12-Pad1)
- U6 pad 3: Net-(R8-Pad2) -> Net-(R12-Pad1)
Routing:
- net GND: track 110.6 -> 55.1 mm, vias 13 -> 9
- net +12V: track 28.5 -> 52.3 mm
- net Net-(SW3-Pad1): track 26.7 -> 17.7 mm
- net /batt_status: track 119.0 -> 127.3 mm
- net Net-(SW5-Pad1): track 37.0 -> 29.2 mm
- net Net-(SW4-Pad1): track 17.4 -> 10.3 mm
- net +3V3: track 113.1 -> 107.1 mm
- net Net-(R12-Pad1): track 0.00 -> 5.29 mm
- net Net-(SW2-Pad1): track 26.1 -> 22.1 mm
- net Net-(D1-Pad2): track 8.64 -> 12.6 mm
- net Net-(R8-Pad2): track 5.32 -> 1.60 mm
- net /RS232/RS232_TX: track 17.5 -> 14.4 mm
- net /charger/BAT-: track 68.3 -> 65.2 mm
- net Net-(D4-Pad2): track 7.79 -> 10.8 mm
- net Net-(R1-Pad2): track 3.34 -> 6.03 mm
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- added copper zone on F.Cu, net +5V
Other:
- board text added: "ON"

Commit message: generando gerbers
Parts:
- added JP2: Jumper_2_Open, Jumper:SolderJumper-2_P1.3mm_Open_TrianglePad1.0x1.5mm, B.Cu at (156.6, 87.1)
- added R13: 10k, Resistor_SMD:R_0603_1608Metric_Pad0.98x0.95mm_HandSolder, B.Cu at (154.4, 87.1)
- added R14: 10k, Resistor_SMD:R_0603_1608Metric_Pad0.98x0.95mm_HandSolder, B.Cu at (154.4, 83.7)
- added R15: 10k, Resistor_SMD:R_0603_1608Metric_Pad0.98x0.95mm_HandSolder, F.Cu at (154.8, 103.4)
- added R16: 10k, Resistor_SMD:R_0603_1608Metric_Pad0.98x0.95mm_HandSolder, F.Cu at (135.3, 102.8)
- added R17: 10k, Resistor_SMD:R_0603_1608Metric_Pad0.98x0.95mm_HandSolder, F.Cu at (135.3, 104.4)
- added R18: 10k, Resistor_SMD:R_0603_1608Metric_Pad0.98x0.95mm_HandSolder, F.Cu at (139.3, 103.8)
- added kibuzzard-629C15DA: G***, kibuzzard-629C15DA, B.Cu at (161.6, 87.1)
Connections:
- C5 pad 1: /batt_status -> /charger/STEP-UP2/VIN
- C6 pad 1: /batt_status -> /charger/STEP-UP2/VIN
- C8 pad 1: /batt_status -> /charger/STEP-UP2/VIN
- L2 pad 1: /batt_status -> /charger/STEP-UP2/VIN
- R7 pad 2: /batt_status -> /charger/STEP-UP2/VIN
- SW1 pad 2: /batt_status -> /charger/STEP-UP2/VIN
- U2 pad 5: /batt_status -> /charger/STEP-UP2/VIN
- U4 pad 3: /batt_status -> /charger/STEP-UP2/VIN
- U5 pad 13: /batt_status -> Net-(U5-Pad13)
- U6 pad 4: /batt_status -> /charger/STEP-UP2/VIN
- U6 pad 5: /batt_status -> /charger/STEP-UP2/VIN
Routing:
- net /batt_status: track 127.3 -> 3.21 mm, vias 3 -> 0
- net /charger/STEP-UP2/VIN: track 0.00 -> 114.9 mm, vias 0 -> 3
- net +3V3: track 107.1 -> 146.4 mm, vias 5 -> 7
- net Net-(U5-Pad13): track 0.00 -> 16.4 mm, vias 0 -> 2
- net /ESP32/UART_RX_0: track 33.9 -> 32.5 mm
- net Net-(U5-Pad36): track 17.7 -> 19.0 mm, vias 1 -> 2
- net /ESP32/UART_TX_0: track 35.5 -> 34.2 mm
- net +12V: track 52.3 -> 51.1 mm
