File: gpsOled.kicad_sch (KiCad schematic)
At the start: 5 parts

Commit message: parcialmente terminada PCB falta verificar tamano de componentes
Parts:
- added H1, H2, H3: MountingHole, MountingHole:MountingHole_3.2mm_M3_DIN965_Pad, symbol Mechanical:MountingHole
- added J4: SSD1306, MSS_Devices:128x64OLED, symbol Connector_Generic:Conn_01x04
- J1: value (none) -> USB_B_Micro; footprint (none) -> Connector_USB:USB_Micro-B_Molex_47346-0001
- J3: value (none) -> Conn_01x03; footprint (none) -> Connector_PinHeader_2.54mm:PinHeader_1x03_P2.54mm_Horizontal
- J5: renamed from J4; value (none) -> RJ45; footprint (none) -> Connector_RJ:RJ45_Amphenol_54602-x08_Horizontal
- J6: renamed from J5; value (none) -> Conn_01x04; footprint (none) -> Connector_PinHeader_2.54mm:PinHeader_1x04_P2.54mm_Horizontal
Connections:
- net +3V3: now also J4.1 (Pin_1)
- net +5V: no longer J1.1 (VBUS)
- net ESP32/SCL: now also J4.3 (Pin_3)
- net ESP32/SDA: now also J4.2 (Pin_2)
- net ESP32/UART_RX_0: now also J3.3 (Pin_3); no longer J3.2 (Pin_2)
- net ESP32/UART_RX_2: now also J6.2 (Pin_2); no longer J6.3 (Pin_3)
- net ESP32/UART_TX_0: now also J3.2 (Pin_2); no longer J3.3 (Pin_3)
- net ESP32/UART_TX_2: now also J6.3 (Pin_3); no longer J6.2 (Pin_2)
- net GND: now also J4.4 (Pin_4)
- net charger/BAT+: now also J2.2 (Pin_2); no longer J2.1 (Pin_1)
- net charger/BAT-: now also J2.1 (Pin_1); no longer J2.2 (Pin_2)
- new net charger/VBUS: J1.1 (VBUS)
Other:
- removed sheet OLED-SSD1306
- sheet ESP32 ports: added status_batt; removed VIN_3V3
- sheet charger: file charger.kicad_sch -> cargador/cargadorDeBateriasLitIon.kicad_sch
- sheet charger ports: added batt_status; removed none
- note added: "STEP-UP 5V TO 12V"
- note removed: "OLED"
- note removed: "STEP-UP"
- title: (none) -> GPS_CHECK
- moved on the sheet: J1, J2

Commit message: terminando, aun falta una ultima revision previa a la fabricacion
Parts:
- H1, H2: footprint MountingHole:MountingHole_3.2mm_M3_DIN965_Pad -> MountingHole:MountingHole_3.2mm_M3_DIN965
- H3: footprint MountingHole:MountingHole_3.2mm_M3_DIN965_Pad -> MountingHole:MountingHole_3.2mm_M3
- J2: value (none) -> Conn_01x02; footprint (none) -> Connector_PinHeader_1.27mm:PinHeader_1x02_P1.27mm_Vertical
- J5: footprint Connector_RJ:RJ45_Amphenol_54602-x08_Horizontal -> MSS_Connector:RJ45_GEN_ZQP_Horizontal
