File: cargador/cargadorDeBateriasLitIon.kicad_sch (KiCad schematic)
At the start: 17 parts, among them Q1 FS8205A, SW1 on/off, U2 TP4056, U3 DW01A, U4 AP1117-33

Commit message: terminando, aun falta una ultima revision previa a la fabricacion
Parts:
- SW1: footprint Button_Switch_THT:SW_CuK_JS202011AQN_DPDT_Angled -> Button_Switch_SMD:SW_SPDT_PCM12
Changed lines of the file:
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@@
       (effects (font (size 1.27 1.27)) (justify left))
     )
-    (property "Footprint" "Button_Switch_THT:SW_CuK_JS202011AQN_DPDT_Angled" (id 2) (at 160.02 66.04 0)
+    (property "Footprint" "Button_Switch_SMD:SW_SPDT_PCM12" (id 2) (at 160.02 66.04 0)
       (effects (font (size 1.27 1.27)) hide)
     )

Commit message: generando gerbers
Parts:
- added JP2: Jumper_2_Open, Jumper:SolderJumper-2_P1.3mm_Open_TrianglePad1.0x1.5mm, symbol Jumper:Jumper_2_Open
Connections:
- net batt_status: now also JP2.2 (B); no longer C5.1, C6.1, R7.2, SW1.2 (B), U2.5 (BAT), U4.3 (VI)
- new net STEP-UP2/VIN: C5.1, C6.1, JP2.1 (A), R7.2, SW1.2 (B), U2.5 (BAT), U4.3 (VI)
Changed lines of the file:
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@@
     (stroke (width 0) (type default) (color 0 0 0 0))
   )
-  (wire (pts (xy 170.18 69.85) (xy 170.18 73.66))
+  (wire (pts (xy 170.18 67.31) (xy 170.18 73.66))
     (stroke (width 0) (type default) (color 0 0 0 0))
   )
@@
     (stroke (width 0) (type default) (color 0 0 0 0))
   )
-  (wire (pts (xy 179.07 69.85) (xy 170.18 69.85))
-    (stroke (width 0) (type default) (color 0 0 0 0))
-  )
   (wire (pts (xy 115.57 107.95) (xy 115.57 116.84))
     (stroke (width 0) (type default) (color 0 0 0 0))
@@
     (stroke (width 0) (type default) (color 0 0 0 0))
   )
+  (wire (pts (xy 182.88 67.31) (xy 185.42 67.31))
+    (stroke (width 0) (type default) (color 0 0 0 0))
+  )
   (wire (pts (xy 160.02 73.66) (xy 160.02 76.2))
     (stroke (width 0) (type default) (color 0 0 0 0))
@@
   )
   (wire (pts (xy 147.32 97.79) (xy 151.13 97.79))
+    (stroke (width 0) (type default) (color 0 0 0 0))
+  )
+  (wire (pts (xy 172.72 67.31) (xy 170.18 67.31))
     (stroke (width 0) (type default) (color 0 0 0 0))
   )
@@
     (effects (font (size 1.27 1.27)) (justify left))
   )
-  (hierarchical_label "batt_status" (shape output) (at 179.07 69.85 0)
+  (hierarchical_label "batt_status" (shape output) (at 185.42 67.31 0)
     (effects (font (size 1.27 1.27)) (justify left))
   )
@@
     (pin "4")
   )
+  (symbol (lib_id "Jumper:Jumper_2_Open") (at 177.8 67.31 0) (unit 1)
+    (in_bom yes) (on_board yes) (fields_autoplaced)
+    (property "Reference" "JP2" (id 0) (at 177.8 60.96 0))
+    (property "Value" "Jumper_2_Open" (id 1) (at 177.8 63.5 0))
+    (property "Footprint" "Jumper:SolderJumper-2_P1.3mm_Open_TrianglePad1.0x1.5mm" (id 2) (at 177.8 67.31 0)
+      (effects (font (size 1.27 1.27)) hide)
+    )
+    (property "Datasheet" "~" (id 3) (at 177.8 67.31 0)
+      (effects (font (size 1.27 1.27)) hide)
+    )
+    (pin "1")
+    (pin "2")
+  )
   (symbol (lib_id "Device:R") (at 48.26 83.82 180) (unit 1)
